File: PCB/DuoSix2.kicad_sch (KiCad schematic)
At the start: 33 parts, among them J1 OLED_DISPLAY, SW1 SW_Push_45deg, SW2 SW_Push_45deg, SW3 SW_Push_45deg, SW4 SW_Push_45deg, SW5 SW_Push_45deg, SW6 SW_Push_45deg, SW7 RotaryEncoder_Switch, SW8 RotaryEncoder_Switch, U1 MOUDLE-SEEEDUINO-XIAO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

Commit message: Altered Design
Removed decoupling capacitors and IC socket to reduce production cost
Parts:
- removed C1, C2, C3, C4, C5, C6, C7, C8: 0.1 μF, 0.1 uF Ceramic Capacitor Through Hole:CAP_Z5UH6UJ5R_VIS, symbol Device:C
